Commit message: update readme and add dependencies

File: turtlebot3/turtlebot3_description/urdf/turtlebot3_burger.urdf.xacro (robot description, xacro)
@@ -140,20 +140,3 @@
     </inertial>
   </link>
-  <xacro:include filename="$(find realsense2_description)/urdf/_d435.urdf.xacro" />
-  <joint name="camera_joint" type="fixed">
-    <origin xyz="0.0 0 0.1" rpy="0 0 0"/>
-    <parent link="base_link"/>
-    <child link="camera_link"/>
-  </joint>
-  <link name="camera_link">
-    <collision>
-      <origin xyz="0.00 0 0" rpy="0 0 0"/>
-      <geometry>
-        <box size="0 0 0"/>
-      </geometry>
-    </collision>
-  </link>
-  <sensor_d435 parent="camera_link" name="robot_camera">
-      <origin xyz="0 0 0" rpy="0 0 0"/>
-  </sensor_d435>
 </robot>
